File: hardware/tinyPPS.kicad_sch (KiCad schematic)
At the start: 68 parts, among them IC1 AP2205-33Y-13, IC2 AP33772SDKZ-13-FA01, J1 USB_C_Receptacle_USB2.0_14P, J2 187-3802, J3 187-3802, J5 SM03B-SRSS-TB_LF__SN_, Q1 DMN3009SFG-7, Q2 DMN3009SFG-7, Q3 BSS123, Q4 BSS123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

Commit message: Remove LED connection and update PD_INT level shifter
Parts:
- removed Q5, Q6: BSS123, Package_TO_SOT_SMD:SOT-23, symbol Transistor_FET:BSS123
- removed R11, R23: 0R, Resistor_SMD:R_0402_1005Metric, symbol Device:R
- removed R19, R20: 10k, Resistor_SMD:R_0402_1005Metric, symbol Device:R
- R9: value 10k -> 5k1
Connections:
- net +3V3: no longer R9.1
- net +5V: no longer R10.1
- net GND: now also R10.2
- net PD_INT: now also R10.1
- net PD_INT_5V: now also IC2.9 (INT), R9.1; no longer R10.2
- net PD_LED: no longer names the net of U1.29 (GPIO18)
- no-connect marks 34 -> 36
Other:
- note added: "5V to 3V3 level shifters"
- note removed: "5V to 3V3 bidirectional level shifters"
- moved on the sheet: R10, R9

Commit message: Use back-to-back N MOS switch with common source
Parts:
- added R11: 10R, Resistor_SMD:R_0402_1005Metric, symbol Device:R
- R3: value 27R -> 100R
Connections:
- net VIN+: now also Q2.5 (D_1), Q2.6 (D_2), Q2.7 (D_3), Q2.8 (D_4), Q2.9 (D_5); no longer Q2.1 (S_1), Q2.2 (S_2), Q2.3 (S_3)
- net at Q1.4 (G), Q2.4 (G): now also R11.1; no longer IC2.23 (PWR_EN)
- net at Q1.5 (D_1), Q1.6 (D_2), Q1.7 (D_3)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: now also IC2.24 (VCC), R6.2; no longer Q2.5 (D_1), Q2.6 (D_2), Q2.7 (D_3), Q2.8 (D_4), Q2.9 (D_5)
- net at Q1.1 (S_1), Q1.2 (S_2), Q1.3 (S_3): now also Q2.1 (S_1), Q2.2 (S_2), Q2.3 (S_3); no longer IC2.24 (VCC), R6.2
- new net: IC2.23 (PWR_EN), R11.2
Other:
- note added: "Back-to-back N-MOS switch in common source configuration"
- note added: "Bidirectional level shifters for I2C pins"
- note added: "DN and DP are not connected, these pins are used for moisture detection"
- note added: "INT can be useful for catching interrupts like OTP, OCP, OVP, UVP, ... HIGH -> interrupt occured"
- note added: "NC pins are passthrough"
- note added: "Not interested in LED indication"
- note added: "Schematic is copy/pasted from RP2040 reference design document"
- note added: "Simple voltage divider is enough to work as an unidirectional level shifter for the PD_INT output pin"
- note added: "Slave address: 0x40"
- note added: "There is no need to add pull up resistors since the OLED has them"
- note added: "min 0.5W 1206"
- note removed: "Slave address 1000000 (0x40)"
- note removed: "There is no need to add pull up resistors since the oled has them"
- moved on the sheet: C1, C2, C22, C3, C4, C5, C6, C7, D1, D2, IC1, IC2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

Commit message: Change rotary encoder to a horizontal type
- Re-route the PCB
- Make PCB with smaller (60mm)
Parts:
- SW1: footprint Rotary_Encoder:RotaryEncoder_Alps_EC11E-Switch_Vertical_H20mm -> Rotary_Encoder:EC11 horizontal
Changed lines of the file:
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@@
 			)
 		)
-		(property "Footprint" "Rotary_Encoder:RotaryEncoder_Alps_EC11E-Switch_Vertical_H20mm"
+		(property "Footprint" "Rotary_Encoder:EC11 horizontal"
 			(at 374.65 191.516 0)
 			(effects

Commit message: Update PCB routing - use +3v3 and GND planes
Parts:
- removed C4: 10u, Capacitor_SMD:C_1206_3216Metric, symbol Device:C
- added C23, C24: 100n, Capacitor_SMD:C_0402_1005Metric, symbol Device:C
Connections:
- net GND: now also C23.2, C24.2
- net VBUS: now also C23.1
- net VBUS_PD: now also C24.1
Other:
- note added: "put as close as possible to the USB connector"
- moved on the sheet: C1, C5, C6, C7, D1, IC2, Q1, Q2, R11, R17, R18, R24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

Commit message: Update schematic with output capacitors
- Add x5 10uF and x1 100uF capacitors to the output
- Move INA226 to be after output capacitors to measure the load and not current of charging capacitors
Parts:
- removed C24: 100n, Capacitor_SMD:C_0402_1005Metric, symbol Device:C
- added C24: 100u, Capacitor_SMD:CP_Elec_6.3x7.7, symbol Device:C_Polarized
- added C25, C26, C27, C4: 10u, Capacitor_SMD:C_1206_3216Metric, symbol Device:C
- added C29: 100n, Capacitor_SMD:C_0402_1005Metric, symbol Device:C
Connections:
- net GND: now also C24.2, C25.2, C26.2, C27.2, C29.1, C4.2
- net PD_INT: now also U1.35 (GPIO23); no longer U1.28 (GPIO17)
- net VBUS_PD: no longer C1.1
- net VIN+: now also C1.1, C24.1, C25.1, C26.1, C27.1, C4.1
- net at Q1.4 (G), Q2.4 (G), R11.1: now also C29.2
Other:
- moved on the sheet: C1, C22, C23, D1, R11, R24, R6, U4
